Commit message: lio-sam

File: launch/include/config/robot.urdf.xacro (robot description, xacro)
@@ -1,4 +1,5 @@
 <?xml version="1.0"?>
 <robot name="lio" xmlns:xacro="http://tixiaoshan.github.io/">
+  <xacro:arg name="namespace" default="jackal1" />
   <xacro:property name="PI" value="3.1415926535897931" />
   <link name="chassis_link"></link>
@@ -15,8 +16,19 @@
     <origin xyz="0 0 0" rpy="0 0 0" />
   </joint>
-  <link name="velodyne"> </link>
-  <joint name="velodyne_joint" type="fixed">
-    <parent link="chassis_link" />
-    <child link="velodyne" />
+   <!-- Velodyne mount stuff -->
+   <link name="velodyne_mount">
+    <visual>
+      <origin xyz="0 0 0.2" rpy="0.0 0.0 0.0" />
+      <geometry>
+        <mesh filename="$(find jackal_description)/meshes/velodyne_tower.stl"/>
+      </geometry>
+      <material name="aluminum" >
+        <color rgba="0.45 0.45 0.45 1"/>
+      </material>
+    </visual>
+  </link>
+  <joint name="velodyne_mount_joint" type="fixed">
+    <parent link="base_link" />
+    <child link="velodyne_mount" />
     <origin xyz="0 0 0" rpy="0 0 0" />
   </joint>
